File: plate/v1.3-plate-chukozor/chocofi-switch_plate.kicad_sch (KiCad schematic)
At the start: 85 parts, among them J1 MJ-4PP-9, J2 Conn_01x05, J3 Conn_01x02_Female, SW1 SW_SPDT, SW10 SW_PUSH, SW11 SW_PUSH, SW12 SW_PUSH, SW13 RotaryEncoder_Switch, SW14 SW_PUSH, SW15 SW_PUSH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

Commit message: wip
Parts:
- SW10, SW11, SW12, SW14, SW15, SW16, SW17, SW18, SW19, SW2, SW20, SW21, SW22, SW23, SW24, SW25, SW3, SW4, SW5, SW6, SW8, SW9: footprint keyswitches:Kailh_socket_PG1350_reversible -> Switch_plate_Chukozor:Chukozor_switch_plate-Khail_chocv1
Changed lines of the file:
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@@
 			)
 		)
-		(property "Footprint" "keyswitches:Kailh_socket_PG1350_reversible"
+		(property "Footprint" "Switch_plate_Chukozor:Chukozor_switch_plate-Khail_chocv1"
 			(at 58.42 26.67 0)
 			(effects
@@
 			)
 		)
-		(property "Footprint" "keyswitches:Kailh_socket_PG1350_reversible"
+		(property "Footprint" "Switch_plate_Chukozor:Chukozor_switch_plate-Khail_chocv1"
 			(at 76.2 26.67 0)
 			(effects
@@
 			)
 		)
-		(property "Footprint" "keyswitches:Kailh_socket_PG1350_reversible"
+		(property "Footprint" "Switch_plate_Chukozor:Chukozor_switch_plate-Khail_chocv1"
 			(at 93.98 26.67 0)
 			(effects
@@
 			)
 		)
-		(property "Footprint" "keyswitches:Kailh_socket_PG1350_reversible"
+		(property "Footprint" "Switch_plate_Chukozor:Chukozor_switch_plate-Khail_chocv1"
 			(at 111.76 26.67 0)
 			(effects
@@
 			)
 		)
-		(property "Footprint" "keyswitches:Kailh_socket_PG1350_reversible"
+		(property "Footprint" "Switch_plate_Chukozor:Chukozor_switch_plate-Khail_chocv1"
 			(at 129.54 26.67 0)
 			(effects
@@
 			)
 		)
-		(property "Footprint" "keyswitches:Kailh_socket_PG1350_reversible"
+		(property "Footprint" "Switch_plate_Chukozor:Chukozor_switch_plate-Khail_chocv1"
 			(at 58.42 41.91 0)
 			(effects
@@
 			)
 		)
-		(property "Footprint" "keyswitches:Kailh_socket_PG1350_reversible"
+		(property "Footprint" "Switch_plate_Chukozor:Chukozor_switch_plate-Khail_chocv1"
 			(at 76.2 41.91 0)
 			(effects
@@
 			)
 		)
-		(property "Footprint" "keyswitches:Kailh_socket_PG1350_reversible"
+		(property "Footprint" "Switch_plate_Chukozor:Chukozor_switch_plate-Khail_chocv1"
 			(at 93.98 41.91 0)
 			(effects
@@
 			)
 		)
-		(property "Footprint" "keyswitches:Kailh_socket_PG1350_reversible"
+		(property "Footprint" "Switch_plate_Chukozor:Chukozor_switch_plate-Khail_chocv1"
 			(at 111.76 41.91 0)
 			(effects
@@
 			)
 		)
-		(property "Footprint" "keyswitches:Kailh_socket_PG1350_reversible"
+		(property "Footprint" "Switch_plate_Chukozor:Chukozor_switch_plate-Khail_chocv1"
 			(at 129.54 41.91 0)
 			(effects
@@
 			)
 		)
-		(property "Footprint" "keyswitches:Kailh_socket_PG1350_reversible"
+		(property "Footprint" "Switch_plate_Chukozor:Chukozor_switch_plate-Khail_chocv1"
 			(at 58.42 57.15 0)
 			(effects
@@
 			)
 		)
-		(property "Footprint" "keyswitches:Kailh_socket_PG1350_reversible"
+		(property "Footprint" "Switch_plate_Chukozor:Chukozor_switch_plate-Khail_chocv1"
 			(at 76.2 57.15 0)
 			(effects
@@
 			)
 		)
-		(property "Footprint" "keyswitches:Kailh_socket_PG1350_reversible"
+		(property "Footprint" "Switch_plate_Chukozor:Chukozor_switch_plate-Khail_chocv1"
 			(at 93.98 57.15 0)
 			(effects
@@
 			)
 		)
-		(property "Footprint" "keyswitches:Kailh_socket_PG1350_reversible"
+		(property "Footprint" "Switch_plate_Chukozor:Chukozor_switch_plate-Khail_chocv1"
 			(at 111.76 57.15 0)
 			(effects
@@
 			)
 		)
-		(property "Footprint" "keyswitches:Kailh_socket_PG1350_reversible"
+		(property "Footprint" "Switch_plate_Chukozor:Chukozor_switch_plate-Khail_chocv1"
 			(at 129.54 57.15 0)
 			(effects
@@
 			)
 		)
-		(property "Footprint" "keyswitches:Kailh_socket_PG1350_reversible"
+		(property "Footprint" "Switch_plate_Chukozor:Chukozor_switch_plate-Khail_chocv1"
 			(at 111.76 72.39 0)
 			(effects
@@
 			)
 		)
-		(property "Footprint" "keyswitches:Kailh_socket_PG1350_reversible"
+		(property "Footprint" "Switch_plate_Chukozor:Chukozor_switch_plate-Khail_chocv1"
 			(at 129.54 72.39 0)
 			(effects
@@
 			)
 		)
-		(property "Footprint" "keyswitches:Kailh_socket_PG1350_reversible"
+		(property "Footprint" "Switch_plate_Chukozor:Chukozor_switch_plate-Khail_chocv1"
 			(at 93.98 72.39 0)
 			(effects
@@
 			)
 		)
-		(property "Footprint" "keyswitches:Kailh_socket_PG1350_reversible"
+		(property "Footprint" "Switch_plate_Chukozor:Chukozor_switch_plate-Khail_chocv1"
 			(at 40.64 41.91 0)
 			(effects
@@
 			)
 		)
-		(property "Footprint" "keyswitches:Kailh_socket_PG1350_reversible"
+		(property "Footprint" "Switch_plate_Chukozor:Chukozor_switch_plate-Khail_chocv1"
 			(at 40.64 26.67 0)
 			(effects
@@
 			)
 		)
-		(property "Footprint" "keyswitches:Kailh_socket_PG1350_reversible"
+		(property "Footprint" "Switch_plate_Chukozor:Chukozor_switch_plate-Khail_chocv1"
 			(at 40.64 57.15 0)
 			(effects
@@
 			)
 		)
-		(property "Footprint" "keyswitches:Kailh_socket_PG1350_reversible"
+		(property "Footprint" "Switch_plate_Chukozor:Chukozor_switch_plate-Khail_chocv1"
 			(at 76.2 72.39 0)
 			(effects
