File: pcb/hotswap/chocofi.kicad_pcb (KiCad board)
At the start: 2 copper layers, 152.9 x 103.1 mm, 52 parts, among them J1 MJ-4PP-9, J2 Conn_01x05, SW1 SW_Chuk, SW10 SW_Chuk, SW11 SW_Chuk, SW12 SW_Chuk, SW13 SW_Chuk, SW14 SW_Chuk, SW15 SW_Chuk, SW16 SW_Chuk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

Commit message: wip
Parts:
- removed JP1, JP10: SDA, kbd:Jumper
- removed JP2, JP9: CS, kbd:Jumper
- removed JP3, JP8: SCL, kbd:Jumper
- removed JP4, JP7: GND, kbd:Jumper
- removed JP5, JP6: VCC, kbd:Jumper
- J2: value Conn_01x05 -> Conn_01x04; footprint nice_view:nice_view_1side -> Switches_Chukozor:oled_display_Chukozor
- SB1: value SolderJumper_3_Open -> switches_oled_display; footprint cornia-footprints:SolderJumper-3_I2C -> Switches_Chukozor:switches_oled_display
- SB2: footprint cornia-footprints:SolderJumper-3_I2C -> Switches_Chukozor:SolderJumper-3_I2C_Chukozor
- SW14, SW19, SW2, SW8: footprint Switches_Chukozor:Kailh_socket_PG1350_reversible_Chukozor_shortenedbis -> Switches_Chukozor:Kailh_socket_PG1350_reversible_Chukozor
- moved Handedness1 29.8 mm to (178.2, 100.4)
- moved SB1 22.8 mm to (184.7, 90.8)
- moved H1 19.5 mm to (3.41, 21.9)
- moved H3 19.5 mm to (3.41, 27.9)
- moved SB2 18.3 mm to (185.9, 68.7), turned to 90 degrees
- moved J1 13.8 mm to (201.7, 108.0)
- moved J2 12.1 mm to (184.7, 93.7)
- moved RSW1 10.0 mm to (195.9, 96.9)
- moved U1 6.00 mm to (186.4, 69.9)
- moved R1 1.82 mm to (166.7, 111.4)
- moved R2 1.03 mm to (166.4, 106.7)
- moved SW24 0.56 mm to (125.3, 110.9)
- turned SW1 to 0 degrees
- turned SW13 to 0 degrees
- turned SW19 to 180 degrees
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Connections:
- J2 pad 1: Net-(J2-Pin_1) -> Net-(J2-Pin_4)
- J2 pad 2: Net-(J2-Pin_2) -> Net-(J2-Pin_3)
- J2 pad 3: Net-(J2-Pin_3) -> Net-(J2-Pin_2)
- J2 pad 4: Net-(J2-Pin_4) -> Net-(J2-Pin_1)
- SB1 pad 1: VCC -> Net-(J2-Pin_4)
- SB1 pad 2: VI2C -> Net-(J2-Pin_3)
- SB1 pad 3: VBUS -> Net-(J2-Pin_2)
Other:
- outline, holes or cut-outs redrawn
- board text added: "${REFERENCE}"
- board text removed: "RIGHT HAND"
- board text removed: "SOLDER HERE FOR LEFT SIDE"

Commit message: wip
Parts:
- moved R1 0.35 mm to (166.4, 111.7)
Other:
- outline, holes or cut-outs redrawn
Changed lines of the file:
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@@
 		(allow_soldermask_bridges_in_footprints no)
 		(aux_axis_origin 145.73 12.66)
-		(grid_origin 67.91 73.4)
+		(grid_origin 85.91 104.4)
 		(pcbplotparams
 			(layerselection 0x00010fc_ffffffff)
@@
 		)
 		(fp_text user "3V3"
-			(at -2.8 0 360)
+			(at -2.8 0 0)
 			(layer "F.SilkS")
 			(effects
@@
 		)
 		(fp_text user "5V"
-			(at 2.9 0 360)
+			(at 2.9 0 0)
 			(layer "F.SilkS")
 			(effects
@@
 	(footprint "Resistances_Chukozor:R_0805_double_face_Chukozor"
 		(layer "B.Cu")
-		(at 166.66 111.4 180)
+		(at 166.41 111.65 180)
 		(descr "Resistor SMD 0805 (2012 Metric), square (rectangular) end terminal, IPC_7351 nominal with elongated pad for handsoldering. (Body size source: IPC-SM-782 page 72, https://www.pcb-3d.com/wordpress/wp-content/uploads/ipc-sm-782a_amendment_1_and_2.pdf), generated with kicad-footprint-generator")
 		(tags "resistor handsolder")
@@
 	)
 	(gr_arc
-		(start 75.11 107.4)
-		(mid 76.01 106.5)
-		(end 76.91 107.4)
+		(start 75.161285 113.629813)
+		(mid 75.364373 113.071344)
+		(end 75.91 112.835923)
 		(stroke
 			(width 0.15)
@@
 	)
 	(gr_arc
-		(start 76.91 100.1)
-		(mid 76.01 101)
-		(end 75.11 100.1)
-		(stroke
-			(width 0.15)
-			(type default)
-		)
-		(layer "Edge.Cuts")
-	)
-	(gr_arc
 		(start 202.8 146.6)
 		(mid 202.282843 147.048528)
@@
 	)
 	(gr_line
-		(start 76.91 100.1)
-		(end 76.91 90.5)
-		(stroke
-			(width 0.15)
-			(type default)
-		)
-		(layer "Edge.Cuts")
-	)
-	(gr_line
-		(start 75.11 100.1)
-		(end 75.11 90.5)
-		(stroke
-			(width 0.15)
-			(type default)
-		)
-		(layer "Edge.Cuts")
-	)
-	(gr_line
-		(start 74.41 115.9)
-		(end 59.41 115.9)
+		(start 74.46 115.85)
+		(end 59.42 115.849999)
 		(stroke
 			(width 0.15)
@@
 		(layer "Edge.Cuts")
 	)
-	(gr_line
-		(start 76.91 107.4)
-		(end 76.916573 112.2)
-		(stroke
-			(width 0.15)
-			(type default)
-		)
-		(layer "Edge.Cuts")
-	)
 	(gr_arc
-		(start 59.41 115.9)
-		(mid 59.056447 115.753553)
-		(end 58.91 115.4)
+		(start 59.42 115.849999)
+		(mid 59.061397 115.705644)
+		(end 58.909901 115.35)
 		(stroke
 			(width 0.15)
@@
 	(gr_arc
 		(start 93.220002 112.835923)
-		(mid 93.733256 113.007332)
+		(mid 93.726065 113.015312)
 		(end 93.95706 113.5)
 		(stroke
@@
 		(layer "Edge.Cuts")
 	)
+	(gr_line
+		(start 93.220002 112.835923)
+		(end 75.91 112.835923)
+		(stroke
+			(width 0.15)
+			(type default)
+		)
+		(layer "Edge.Cuts")
+	)
 	(gr_arc
-		(start 77.51 112.793427)
-		(mid 77.090384 112.619616)
-		(end 76.916573 112.2)
+		(start 75.986189 114.069616)
+		(mid 76.16 113.65)
+		(end 76.579616 113.476189)
 		(stroke
 			(width 0.15)
@@
 	)
 	(gr_line
-		(start 75.11 83.2)
-		(end 75.11 73.5)
+		(start 75.161285 113.629813)
+		(end 75.16 115.15)
 		(stroke
 			(width 0.15)
@@
 		(layer "Edge.Cuts")
 	)
-	(gr_arc
-		(start 75.11 90.5)
-		(mid 76.01 89.6)
-		(end 76.91 90.5)
+	(gr_line
+		(start 75.11 83.2)
+		(end 75.11 73.5)
 		(stroke
 			(width 0.15)
@@
 	)
 	(gr_arc
-		(start 75.11 115.2)
-		(mid 74.904975 115.694975)
-		(end 74.41 115.9)
+		(start 75.16 115.15)
+		(mid 74.954975 115.644975)
+		(end 74.46 115.85)
 		(stroke
 			(width 0.15)
@@
 	(gr_line
 		(start 58.91 65.4)
-		(end 58.91 115.4)
+		(end 58.909901 115.35)
 		(stroke
 			(width 0.15)
@@
 		)
 		(layer "Edge.Cuts")
-	)
-	(gr_line
-		(start 77.51 112.793427)
-		(end 93.21 112.835923)
-		(stroke
-			(width 0.15)
-			(type solid)
-		)
-		(layer "Edge.Cuts")

Commit message: wip
Parts:
- J1: footprint kbd:MJ-4PP-9 -> Switches_Chukozor:MJ-4PP-9_Chukozor
- moved J1 6.21 mm to (195.5, 107.2), turned to 0 degrees
Routing:
- net VCC: track 0.00 -> 5.97 mm
Other:
- board size 152.9 x 103.1 mm -> 152.9 x 103 mm

Commit message: wip
Connections:
- U1 pad 30: RAW -> VBUS

Commit message: wip
Parts:
- added C1: 1uF, cornia-footprints:C_0805, F.Cu at (206.8, 104.0)
- added J3: Conn_01x04, Switches_Chukozor:oled_display_Chukozor, F.Cu at (184.4, 93.0)
- J1: value MJ-4PP-9 -> Conn_01x01_Pin; footprint Switches_Chukozor:MJ-4PP-9_Chukozor -> cornia-footprints:1Pin
- J2: value Conn_01x04 -> MJ-4PP-9; footprint Switches_Chukozor:oled_display_Chukozor -> Switches_Chukozor:MJ-4PP-9_Chukozor
- SW1, SW13, SW7: footprint Switches_Chukozor:Kailh_socket_PG1350_reversible_Chukozor_shortenedbis -> Switches_Chukozor:Kailh_socket_PG1350_reversible_Chukozor_shortened_LED
- SW10, SW11, SW12, SW16, SW17, SW18, SW19, SW20, SW21, SW22, SW23, SW4, SW5, SW6: footprint Switches_Chukozor:Kailh_socket_PG1350_reversible_Chukozor -> Switches_Chukozor:Kailh_socket_PG1350_reversible_Chukozor_LED
- SW14, SW2, SW8: footprint Switches_Chukozor:Kailh_socket_PG1350_reversible_Chukozor -> Switches_Chukozor:Kailh_socket_PG1350_reversible_Chukozor_Col_5_LED
- SW15, SW9: footprint Switches_Chukozor:Kailh_socket_PG1350_reversible_Chukozor -> Switches_Chukozor:Kailh_socket_PG1350_reversible_Chukozor_Top_Col_4_LED
- SW3: footprint Switches_Chukozor:Kailh_socket_PG1350_reversible_Chukozor_shortenedbis -> Switches_Chukozor:Kailh_socket_PG1350_reversible_Chukozor_Top_Col_4_shortened_LED
- moved J1 130.5 mm to (71.7, 65.8)
- moved H8 112.7 mm to (3.81, 34.6)
- moved H6 14.0 mm to (193.9, 120.0)
- moved J2 13.0 mm to (195.5, 100.9)
- moved Handedness1 5.47 mm to (173.1, 98.3)
- moved RSW1 1.92 mm to (197.8, 96.6)
- moved SB1 0.68 mm to (184.5, 90.2)
Connections:
- SB1 pad 1: Net-(J2-Pin_4) -> Net-(J3-Pin_4)
- SB1 pad 2: Net-(J2-Pin_3) -> Net-(J3-Pin_3)
- SB1 pad 3: Net-(J2-Pin_2) -> Net-(J3-Pin_2)
- SB1 pad 4: Net-(J2-Pin_1) -> Net-(J3-Pin_1)
Other:
- outline, holes or cut-outs redrawn
- board text removed: "BAT"
- board text removed: "RST"
- board text removed: "SCL"
- board text removed: "SDA"

Commit message: wip
Parts:
- moved SW19 140.4 mm to (103.9, 109.4), turned to 0 degrees
- moved SW20 46.3 mm to (139.2, 139.3)
Connections:
- SW11 pad 5: Net-(SW10-DIN) -> Net-(SW11-DOUT)
- SW11 pad 7: Net-(SW11-DIN) -> Net-(SW10-DOUT)
- SW12 pad 5: Net-(SW11-DIN) -> Net-(SW12-DOUT)
- SW12 pad 7: Net-(SW12-DIN) -> Net-(SW11-DOUT)
- SW13 pad 5: Net-(SW12-DIN) -> Net-(SW13-DOUT)
- SW19 pad 5: Net-(SW18-DIN) -> Net-(SW19-DOUT)
- SW19 pad 7: Net-(SW19-DIN) -> LED
- SW20 pad 5: Net-(SW19-DIN) -> Net-(SW20-DOUT)
- SW20 pad 7: Net-(SW20-DIN) -> Net-(SW19-DOUT)
- SW21 pad 5: Net-(SW20-DIN) -> Net-(SW21-DOUT)
- SW21 pad 7: Net-(SW21-DIN) -> Net-(SW20-DOUT)
- SW22 pad 5: Net-(SW21-DIN) -> Net-(SW22-DOUT)
- SW22 pad 7: Net-(SW22-DIN) -> Net-(SW21-DOUT)
- SW23 pad 5: Net-(SW22-DIN) -> Net-(SW18-DIN)
- SW23 pad 7: LED -> Net-(SW22-DOUT)
- SW6 pad 7: Net-(SW6-DIN) -> Net-(SW12-DOUT)
- SW7 pad 5: Net-(SW6-DIN) -> Net-(SW7-DOUT)
- SW7 pad 7: Net-(SW7-DIN) -> Net-(SW13-DOUT)
- SW8 pad 5: Net-(SW7-DIN) -> Net-(SW8-DOUT)
- SW8 pad 7: Net-(SW8-DIN) -> Net-(SW7-DOUT)
- SW9 pad 5: Net-(SW8-DIN) -> Net-(SW10-DIN)
- SW9 pad 7: Net-(SW10-DOUT) -> Net-(SW8-DOUT)
Routing:
- net row0: track 0.00 -> 145.8 mm
- net row1: track 0.00 -> 113.1 mm
- net row2: track 0.00 -> 110.7 mm
- net col2: track 0.00 -> 53.5 mm
- net col5: track 0.00 -> 37.5 mm
- net col4: track 0.00 -> 35.7 mm
- net col0: track 0.00 -> 35.6 mm
- net col3: track 0.00 -> 35.6 mm
- net col1: track 0.00 -> 35.6 mm
