File: pcb/hotswap/chocofi.kicad_pcb (KiCad board)
At the start: 2 copper layers, 161.6 x 123.9 mm, 77 parts, among them J1 MJ-4PP-9, J2 Conn_01x04, SW1 SW_Chuk, SW10 SW_Chuk, SW11 SW_Chuk, SW12 SW_Chuk, SW13 SW_Chuk, SW14 SW_Chuk, SW15 SW_Chuk, SW16 SW_Chuk, SW17 SW_Chuk, SW18 SW_Chuk, SW19 SW_Chuk, SW2 SW_Chuk, SW20 SW_Chuk, SW21 SW_Chuk, SW22 SW_Chuk, SW23 SW_Chuk, SW24 SW_Chuk, SW25 SW_Chuk, SW26 SW_Chuk, SW27 SW_Chuk, SW28 SW_Chuk, SW29 SW_Chuk, SW3 SW_Chuk, SW30 SW_Chuk, SW4 SW_Chuk, SW5 SW_Chuk, SW6 SW_Chuk, SW7 SW_Chuk, SW8 SW_Chuk, SW9 SW_Chuk, U1 RP2040-ProMicro

Commit message: wip
Parts:
- U1: footprint cornia-footprints:RP2040-ProMicro -> cornia-footprints:RP2040-ProMicro_simplified
Routing:
- net VI2C: track 46.1 -> 43.0 mm
- net SDA: track 43.5 -> 42.3 mm
- net data: track 78.3 -> 77.2 mm

Commit message: Update chocofi.kicad_pcb
Routing:
- net col3: track 187.5 -> 188.1 mm

Commit message: Update chocofi.kicad_pcb
Parts:
- moved ENC1 5.37 mm to (116.5, 139.0)
- moved H4 3.19 mm to (106.4, 126.5)
- moved H5 1.45 mm to (133.8, 126.7)
- moved D12 0.21 mm to (166.0, 76.5)
Routing:
- net col0: track 113.8 -> 246.6 mm, vias 0 -> 1
- net Net-(SW11-DIN): track 28.1 -> 7.75 mm
- net row2: track 129.3 -> 149.0 mm, vias 1 -> 2
- net row1: track 114.9 -> 131.7 mm, vias 0 -> 1
- net ENCA: track 112.0 -> 127.8 mm
- net ENCB: track 108.1 -> 120.9 mm
- net row0: track 108.9 -> 118.2 mm, vias 1 -> 2
- net col5: track 207.6 -> 205.8 mm
- net data: track 77.2 -> 78.3 mm

Commit message: Update chocofi.kicad_pcb
Parts:
- moved H5 4.14 mm to (132.9, 130.7)
- moved H4 3.75 mm to (109.1, 129.1)
- moved Handedness1 0.30 mm to (179.4, 61.5)
Routing:
- net SCL: track 33.6 -> 35.2 mm
- net col3: track 188.4 -> 186.8 mm
- net ENCB: track 120.9 -> 119.9 mm
- net col2: track 208.2 -> 207.3 mm
- net col4: track 169.7 -> 168.9 mm
- net VI2C: track 43.0 -> 42.2 mm
- net ENCA: track 127.8 -> 127.1 mm
- net row1: vias 1 -> 0
Other:
- board text added: "For Trackpad"

Commit message: wip
Parts:
- H2, H4, H5: footprint Mounting_hole_Chukozor:Passthrough_hole_chukozor_M2 -> Mounting_hole_Chukozor:Passthrough_hole_chukozor_M2_Big
- moved H4 84.1 mm to (180.9, 85.4)
- moved H5 1.91 mm to (132.7, 128.8)
Routing:
- net VBUS: track 951.1 -> 949.8 mm
- net ENCA: track 127.1 -> 126.0 mm
- net ENCB: track 119.9 -> 118.8 mm
- net col0: track 246.8 -> 247.7 mm
Other:
- board size 161.6 x 123.9 mm -> 161.7 x 120.6 mm
