File: pcb/hotswap/chocofi.kicad_pcb (KiCad board)
At the start: 2 copper layers, 164.3 x 133.4 mm, 93 parts, among them J2 Conn_01x04, Q1 TIP120, SW1 SW_Chuk, SW10 SW_Chuk, SW11 SW_Chuk, SW12 SW_Chuk, SW13 SW_Chuk, SW14 SW_Chuk, SW15 SW_Chuk, SW16 SW_Chuk, SW17 SW_Chuk, SW18 SW_Chuk, SW19 SW_Chuk, SW2 SW_Chuk, SW20 SW_Chuk, SW21 SW_Chuk, SW22 SW_Chuk, SW23 SW_Chuk, SW24 SW_Chuk, SW25 SW_Chuk, SW26 SW_Chuk, SW27 SW_Chuk, SW28 SW_Chuk, SW29 SW_Chuk, SW3 SW_Chuk, SW30 SW_Chuk, SW4 SW_Chuk, SW5 SW_Chuk, SW6 SW_Chuk, SW7 SW_Chuk, SW8 SW_Chuk, SW9 SW_Chuk, U1 RP2040-ProMicro, U2 TRRS

Commit message: wip
Routing:
- net col5: track 122.1 -> 130.0 mm
- net ENCB: track 119.6 -> 121.0 mm
- net ENCA: track 119.8 -> 120.3 mm
- net VBUS: track 958.3 -> 958.8 mm

Commit message: wip
Parts:
- moved JP1 0.34 mm to (183.5, 109.0)
Routing:
- net col5: track 130.0 -> 168.8 mm, vias 2 -> 3

Commit message: Update chocofi.kicad_pcb
Routing:
- net LED: track 19.6 -> 102.2 mm

Commit message: Update chocofi.kicad_pcb
Routing:
- net (no net): track 8.80 -> 0.00 mm
- net GND-VIK: vias 877 -> 2
- net GND: vias 4 -> 879

Commit message: wip
Routing:
- net col0: track 214.5 -> 253.1 mm, vias 1 -> 3
- net col5: track 168.8 -> 195.8 mm, vias 3 -> 4
