File: pcb/hotswap/chocofi.kicad_sch (KiCad schematic)
At the start: 106 parts, among them J1 Conn_01x03, J2 Conn_01x04, J3 Conn_01x03, K1 FPC_8pins_687108183722, K2 FPC_8pins_687108183722, K3 FPC_8pins_687108183722, K4 FPC_8pins_687108183722, K5 FPC_8pins_687108183722, K6 FPC_8pins_687108183722, Q1 TIP120, SW1 SW_Chuk, SW10 SW_Chuk, SW11 SW_Chuk, SW12 SW_Chuk, SW13 SW_Chuk, SW14 SW_Chuk, SW15 SW_Chuk, SW16 SW_Chuk, SW17 SW_Chuk, SW18 SW_Chuk, SW2 SW_Chuk, SW22 SW_Chuk, SW23 SW_Chuk, SW24 SW_Chuk, SW3 SW_Chuk, SW4 SW_Chuk, SW5 SW_Chuk, SW6 SW_Chuk, SW7 SW_Chuk, SW8 SW_Chuk, SW9 SW_Chuk, U1 RP2040-ProMicro-with-18thgpio, U2 TRRS_Chuck

Commit message: wip
Parts:
- KHigh-1: footprint Switches_Chukozor:FPC_8pins_687108183722 -> FPC_connectors_Chukozor:FPC_8pins_687108183722_reversible-Mobile-IN-TOPP-FROMABOVE
- KLow-1: footprint FPC_connectors_Chukozor:FPC_8pins_687108183722_reversible-Mobile-IN-LOW-V2 -> FPC_connectors_Chukozor:FPC_8pins_687108183722_reversible-Mobile-IN-LOW-FROMBELOW
- KLow-2: footprint FPC_connectors_Chukozor:FPC_8pins_687108183722_reversible-Mobile-IN-LOW-V2-BUT-placed-above -> FPC_connectors_Chukozor:FPC_8pins_687108183722_reversible-Mobile-IN-TOPP-FROMBELOW
Changed lines of the file:
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@@
 			)
 		)
-		(property "Footprint" "Switches_Chukozor:FPC_8pins_687108183722"
+		(property "Footprint" "FPC_connectors_Chukozor:FPC_8pins_687108183722_reversible-Mobile-IN-TOPP-FROMABOVE"
 			(at 241.3 182.804 0)
 			(effects
@@
 			)
 		)
-		(property "Footprint" "FPC_connectors_Chukozor:FPC_8pins_687108183722_reversible-Mobile-IN-LOW-V2"
+		(property "Footprint" "FPC_connectors_Chukozor:FPC_8pins_687108183722_reversible-Mobile-IN-LOW-FROMBELOW"
 			(at 286.258 199.568 0)
 			(effects
@@
 			)
 		)
-		(property "Footprint" "FPC_connectors_Chukozor:FPC_8pins_687108183722_reversible-Mobile-IN-LOW-V2-BUT-placed-above"
+		(property "Footprint" "FPC_connectors_Chukozor:FPC_8pins_687108183722_reversible-Mobile-IN-TOPP-FROMBELOW"
 			(at 191.262 196.266 0)
 			(effects

Commit message: wip
Parts:
- KLow-1: footprint FPC_connectors_Chukozor:FPC_8pins_687108183722_reversible-Mobile-IN-LOW-FROMBELOW -> FPC_connectors_Chukozor:FPC_8pins_687108183722_reversible-Mobile-IN-LOW-V2
- KLow-2: footprint FPC_connectors_Chukozor:FPC_8pins_687108183722_reversible-Mobile-IN-TOPP-FROMBELOW -> FPC_connectors_Chukozor:FPC_8pins_687108183722_reversible-Mobile-IN-LOW-V2
Changed lines of the file:
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@@
 			"AAAAAAAAAAAAAAAAAAAAAAAAAAAAAAAAAAAAAAAAAAAAAAAAAAAAAAAAAAAAAAAAAAAAAAAAAAAA"
 			"AAAAAAAAAAAAAAAAAAAAAAAAAAAAAAAAAAAAAAAAAAAAAAAAAAAAAAAAAAAAAAAAAAAAAAAAAAAA"
+			"AAAAAAAAAAAAAAAAAAAAAAAAAAAAAAAAAAAAAAAAAAAAAAAAAAAAAAAAAAAAAAAAAAAAAAAAAAAA"
+			"AAAAAAAAAAAAAAAAAAAAAAAAAAAAAAAAAAAAAAAAAAAAAAAAAAAAAAAAAAAAAAAAAAAAAAAAAAAA"
+			"AAAAAAAAAAAAAAAAAAAAAAAAAAAAAAAAAAAAAAAAAAAAAAAAAAAAAAAAAAAAAAAAAAAAAAAAAAAA"
+			"AAAAAAAAAAAAAAAAAAAAAAAAAAAAAAAAAAAAAAAAAAAAAAAAAAAAAAAAAAAAAAAAAAAAAAAAAAAA"
+			"AAAAAAAAAAAAAAAAAAAAAAAAAAAAAAAAAAAAAAAAAAAAAAAAAAAAAAAAAAAAAAAAAAAAAAAAAAAA"
+			"AAAAAAAAAAAAAAAAAAAAAAAAAAAAAAAAAAAAAAAAAAAAAAAAAAAAAAAAAAAAAAAAAAAAAAAAAAAA"
+			"AAAAAAAAAAAAAAAAAAAAAAAAAAAAAAAAAAAAAAAAAAAAAAAAAAAAAAAAAAAAAAAAAAAAAAAAAAAA"
+			"AAAAAAAAAAAAAAAAAAAAAAAAAAAAAAAAAAAAAAAAAAAAAAAAAAAAAAAAAAAAAAAAAAAAAAAAAAAA"
+			"AAAAAAAAAAAAAAAAAAAAAAAAAAAAAAAAAAAAAAAAAAAAAAAAAAAAAAAAAAAAAAAAAAAAAAAAAAAA"
+			"AAAAAAAAAAAAAAAAAAAAAAAAAAAAAAAAAAAAAAAAAAAAAAAAAAAAAAAAAAAAAAAAAAAAAAAAAAAA"
+			"AAAAAAAAAAAAAAAAAAAAAAAAAAAAAAAAAAAAAAAAAAAAAAAAAAAAAAAAAAAAAAAAAAAAAAAAAAAA"
+			"AAAAAAAAAAAAAAAAAAAAAAAAAAAAAAAAAAAAAAAAAAAAAAAAAAAAAAAAAAAAAAAAAAAAAAAAAAAA"
+			"AAAAAAAAAAAAAAAAAAAAAAAAAAAAAAAAAAAAAAAAAAAAAAAAAAAAAAAAAAAAAAAAAAAAAAAAAAAA"
+			"AAAAAAAAAAAAAAAAAAAAAAAAAAAAAAAAAAAAAAAAAAAAAAAAAAAAAAAAAAAAAAAAAAAAAAAAAAAA"
+			"AAAAAAAAAAAAAAAAAAAAAAAAAAAAAAAAAAAAAAAAAAAAAAAAAAAAAAAAAAAAAAAAAAAAAAAAAAAA"
+			"AAAAAAAAAAAAAAAAAAAAAAAAAAAAAAAAAAAAAAAAAAAAAAAAAAAAAAAAAAAAAAAAAAAAAAAAAAAA"
+			"AAAAAAAAAAAAAAAAAAAAAAAAAAAAAAAAAAAAAAAAAAAAAAAAAAAAAAAAAAAAAAAAAAAAAAAAAAAA"
+			"AAAAAAAAAAAAAAAAAAAAAAAAAAAAAAAAAAAAAAAAAAAAAAAAAAAAAAAAAAAAAAAAAAAAAAAAAAAA"
 			"AAAAAA=="
 		)
@@
 			)
 		)
-		(property "Footprint" "FPC_connectors_Chukozor:FPC_8pins_687108183722_reversible-Mobile-IN-LOW-FROMBELOW"
+		(property "Footprint" "FPC_connectors_Chukozor:FPC_8pins_687108183722_reversible-Mobile-IN-LOW-V2"
 			(at 286.258 199.568 0)
 			(effects
@@
 		(pin "1"
 		)
-		(pin "osef"
+		(pin "7"
 		)
 		(instances
@@
 			)
 		)
-		(property "Footprint" "FPC_connectors_Chukozor:FPC_8pins_687108183722_reversible-Mobile-IN-TOPP-FROMBELOW"
+		(property "Footprint" "FPC_connectors_Chukozor:FPC_8pins_687108183722_reversible-Mobile-IN-LOW-V2"
 			(at 191.262 196.266 0)
 			(effects
@@
 		(pin "1"
 		)
-		(pin "osef"
+		(pin "7"
 		)
 		(instances

Commit message: wip
Connections:
- net at KHigh-1.1 (Diode2Switch): now also Flick2.2
Changed lines of the file:
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@@
 	(wire
 		(pts
-			(xy 230.378 96.774) (xy 228.854 96.774)
-		)
-		(stroke
-			(width 0)
-			(type default)
-		)
-	)
-	(wire
-		(pts
 			(xy 146.05 223.52) (xy 146.05 203.2)
 		)
@@
 	(wire
 		(pts
+			(xy 228.6 96.774) (xy 230.378 96.774)
+		)
+		(stroke
+			(width 0)
+			(type default)
+		)
+	)
+	(wire
+		(pts
 			(xy 232.156 362.204) (xy 237.998 362.204)
 		)
@@
 			"AAAAAAAAAAAAAAAAAAAAAAAAAAAAAAAAAAAAAAAAAAAAAAAAAAAAAAAAAAAAAAAAAAAAAAAAAAAA"
 			"AAAAAAAAAAAAAAAAAAAAAAAAAAAAAAAAAAAAAAAAAAAAAAAAAAAAAAAAAAAAAAAAAAAAAAAAAAAA"
-			"AAAAAA=="
+			"AAAAAJDcgnH8fwAAAAAAAAAAAADDRe0EUg6UAQAAAAAAAAAA/////wAAAAAAAAAAAAAAAAAAAAAA"
+			"AAAAxcxSgwBCBYCQ3IJx/H8AAAAAAAAAAAAAoiLsBGUhmwEAAAAAAAAAAP////8AAAAAAAAAAAAA"
+			"AAAAAAAAAAAAAPnMboMAQwWAkNyCcfx/AAAAAAAAAAAAAAX45AT5/4oBAAAAAAAAAAD/////AAAA"
+			"AAAAAAAAAAAAAAAAAAAAAAD9zGqDAEQFgJDcgnH8fwAAAAAAAAAAAAASs+YE6emJAQAAAAAAAAAA"
+			"/////wAAAAAAAAAAAAAAAAAAAAAAAAAA8cxmgwBFBYCQ3IJx/H8AAAAAAAAAAAAA+VvpBPn/igEA"
+			"AAAAAAAAAP////8AAAAAAAAAAAAAAAAAAAAAAAAAAPXMYoMARgWAkNyCcfx/AAAAAAAAAAAAAAtK"
+			"7QTn9pMBAAAAAAAAAAD/////AAAAAAAAAAAAAAAAAAAAAAAAAADpzH6DAEcFgJDcgnH8fwAAAAAA"
+			"AAAAAACdWewETkeOAQAAAAAAAAAA/////wAAAAAAAAAAAAAAAAAAAAAAAAAA7cx6gwBIBYCQ3IJx"
+			"/H8AAAAAAAAAAAAAhQvtBLkakAEAAAAAAAAAAP////8AAAAAAAAAAAAAAAAAAAAAAAAAAOHMdoMA"
+			"SQWAkNyCcfx/AAAAAAAAAAAAAGTC5gQ95okBAAAAAAAAAAD/////AAAAAAAAAAAAAAAAAAAAAAAA"
+			"AADlzHKDAEoFgJDcgnH8fwAAAAAAAAAAAABoquwEIRCZAQAAAAAAAAAA/////wAAAAAAAAAAAAAA"
+			"AAAAAAAAAAAAmcwOgwBLBYCQ3IJx/H8AAAAAAAAAAAAApeTqBP/tnQEAAAAAAAAAAP////8AAAAA"
+			"AAAAAAAAAAAAAAAAAAAAAJ3MCoMATAWAkNyCcfx/AAAAAAAAAAAAANOV5QQjPIoBAAAAAAAAAAD/"
+			"////AAAAAAAAAAAAAAAAAAAAAAAAAACRzAaDAE0FgJDcgnH8fwAAAAAAAAAAAABaVO0E/iSSAQAA"
+			"AAAAAAAA/////wAAAAAAAAAAAAAAAAAAAAAAAAAAlcwCgwBOBYCQ3IJx/H8AAAAAAAAAAAAA9unj"
+			"BH67jAEAAAAAAAAAAP////8AAAAAAAAAAAAAAAAAAAAAAAAAAInMHoMATwWAkNyCcfx/AAAAAAAA"
+			"AAAAAPa75AQ1gYsBAAAAAAAAAAD/////AAAAAAAAAAAAAAAAAAAAAAAAAACNzBqDAFAFgJDcgnH8"
+			"fwAAAAAAAAAAAADATOUE0paKAQAAAAAAAAAA/////wAAAAAAAAAAAAAAAAAAAAAAAAAAgcwWgwBR"
+			"BYCQ3A=="
 		)
 	)

Commit message: wip
Parts:
- removed RSW2: RST, cornia-footprints:SW_SMD_4x4mm, symbol chocofi-rescue:SW_PUSH-kbd-corne-light-rescue
- RSW1: footprint cornia-footprints:SW_SMD_4x4mm -> Switches_Chukozor:SW_SMD_4x4mm-reversible(unconnected)
Changed lines of the file:
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@@
 	)
 	(junction
-		(at 445.008 55.88)
-		(diameter 0)
-		(color 0 0 0 0)
-	)
-	(junction
 		(at 539.242 194.818)
 		(diameter 0)
@@
 	)
 	(junction
-		(at 462.788 64.77)
-		(diameter 0)
-		(color 0 0 0 0)
-	)
-	(junction
 		(at 152.908 351.79)
 		(diameter 0)
@@
 	(wire
 		(pts
-			(xy 462.788 64.77) (xy 460.248 64.77)
-		)
-		(stroke
-			(width 0)
-			(type default)
-		)
-	)
-	(wire
-		(pts
 			(xy 491.998 203.454) (xy 492.76 203.454)
 		)
@@
 	(wire
 		(pts
-			(xy 462.788 64.77) (xy 462.788 55.88)
-		)
-		(stroke
-			(width 0)
-			(type default)
-		)
-	)
-	(wire
-		(pts
 			(xy 220.726 421.894) (xy 87.376 421.894)
 		)
@@
 	(wire
 		(pts
-			(xy 445.008 55.88) (xy 445.008 64.77)
-		)
-		(stroke
-			(width 0)
-			(type default)
-		)
-	)
-	(wire
-		(pts
 			(xy 46.482 260.604) (xy 55.88 260.604)
 		)
@@
 	(wire
 		(pts
-			(xy 462.788 66.04) (xy 462.788 64.77)
-		)
-		(stroke
-			(width 0)
-			(type default)
-		)
-	)
-	(wire
-		(pts
 			(xy 164.592 87.884) (xy 163.576 87.884)
 		)
@@
 	(wire
 		(pts
-			(xy 462.788 55.88) (xy 460.248 55.88)
+			(xy 461.264 55.88) (xy 460.248 55.88)
 		)
 		(stroke
@@
 			"AAAAAPa75AQ1gYsBAAAAAAAAAAD/////AAAAAAAAAAAAAAAAAAAAAAAAAACNzBqDAFAFgJDcgnH8"
 			"fwAAAAAAAAAAAADATOUE0paKAQAAAAAAAAAA/////wAAAAAAAAAAAAAAAAAAAAAAAAAAgcwWgwBR"
-			"BYCQ3A=="
+			"BYCQ3AAAAAAAAAAAAAAAAAAAAAAAAAAAAAAAAAAAAAAAAAAAAAAAAAAAAAAAAAAAAAAAAAAAAAAA"
+			"AAAAAAAAAAAAAAAAAAAAAAAAAAAAAAAAAAAAAAAAAAAAAAAAAAAAAAAAAAAAAAAAAAAAAAAAAAAA"
+			"AAAAAAAAAAAAAAAAAAAAAAAAAAAAAAAAAAAAAAAAAAAAAAAAAAAAAAAAAAAAAAAAAAAAAAAAAAAA"
+			"AAAAAAAAAAAAAAAAAAAAAAAAAAAAAAAAAAAAAAAAAAAAAAAAAAAAAAAAAAAAAAAAAAAAAAAAAAAA"
+			"AAAAAAAAAAAAAAAAAAAAAAAAAAAAAAAAAAAAAAAAAAAAAAAAAAAAAAAAAAAAAAAAAAAAAAAAAAAA"
+			"AAAAAAAAAAAAAAAAAAAAAAAAAAAAAAAAAAAAAAAAAAAAAAAAAAAAAAAAAAAAAAAAAAAAAAAAAAAA"
+			"AAAAAAAAAAAAAAAAAAAAAAAAAAAAAAAAAAAAAAAAAAAAAAAAAAAAAAAAAAAAAAAAAAAAAAAAAAAA"
+			"AAAAAAAAAAAAAAAAAAAAAAAAAAAAAAAAAAAAAAAAAAAAAAAAAAAAAAAAAAAAAAAAAAAAAAAAAAAA"
+			"AAAAAAAAAAAAAAAAAAAAAAAAAAAAAAAAAAAAAAAAAAAAAAAAAAAAAAAAAAAAAAAAAAAAAAAAAAAA"
+			"AAAAAAAAAAAAAAAAAAAAAAAAAAAAAAAAAAAAAAAAAAAAAAAAAAAAAAAAAAAAAAAAAAAAAAAAAAAA"
+			"AAAAAAAAAAAAAAAAAAAAAAAAAAAAAAAAAAAAAAAAAAAAAAAAAAAAAAAAAAAAAAAAAAAAAAAAAAAA"
+			"AAAAAAAAAAAAAAAAAAAAAAAAAAAAAAAAAAAAAAAAAAAAAAAAAAAAAAAAAAAAAAAAAAAAAAAAAAAA"
+			"AAAAAAAAAAAAAAAAAAAAAAAAAAAAAAAAAAAAAAAAAAAAAAAAAAAAAAAAAAAAAAAAAAAAAAAAAAAA"
+			"AAAAAAAAAAAAAAAAAAAAAAAAAAAAAAAAAAAAAAAAAAAAAAAAAAAAAAAAAAAAAAAAAAAAAAAAAAAA"
+			"AAAAAAAAAAAAAAAAAAAAAAAAAAAAAAAAAAAAAAAAAAAAAAAAAAAAAAAAAAAAAAAAAAAAAAAAAAAA"
+			"AAAAAAAAAAAAAAAAAAAAAAAAAAAAAAAAAAAAAAAAAAAAAAAAAAAAAAAAAAAAAAAAAAAAAAAAAAAA"
+			"AAAAAAAAAAAAAAAAAAAAAAAAAAAAAAAAAAAAAAAAAAAAAAAAAAAAAAAAAAAAAAAAAAAAAAAAAAAA"
+			"AAAAAAAAAAAAAAAAAAAAAAAAAAAAAAAAAAAAAAAAAAAAAAAAAAAAAAAAAAAAAAAAAAAAAAAAAAAA"
+			"AAAAAA=="
 		)
 	)
@@
 			)
 		)
-		(property "Footprint" "cornia-footprints:SW_SMD_4x4mm"
+		(property "Footprint" "Switches_Chukozor:SW_SMD_4x4mm-reversible(unconnected)"
 			(at 452.628 55.88 0)
 			(effects
@@
 	(symbol
 		(lib_id "chocofi-rescue:GND-power")
-		(at 462.788 66.04 0)
+		(at 461.264 55.88 90)
 		(unit 1)
 		(exclude_from_sim no)
@@
 		(dnp no)
 		(property "Reference" "#PWR015"
-			(at 462.788 72.39 0)
+			(at 467.614 55.88 0)
 			(effects
 				(font
@@
 		)
 		(property "Value" "GND"
-			(at 462.788 69.85 0)
+			(at 465.074 55.88 0)
 			(effects
 				(font
@@
 		)
 		(property "Footprint" ""
-			(at 462.788 66.04 0)
+			(at 461.264 55.88 0)
 			(effects
 				(font
@@
 		)
 		(property "Datasheet" ""
-			(at 462.788 66.04 0)
+			(at 461.264 55.88 0)
 			(effects
 				(font
@@
 		)
 		(property "Description" ""
-			(at 462.788 66.04 0)
+			(at 461.264 55.88 0)
 			(effects
 				(font
@@
 					(unit 1)
 				)
-			)
-		)
-	)
-	(symbol
-		(lib_id "chocofi-rescue:SW_PUSH-kbd-corne-light-rescue")
-		(at 452.628 64.77 0)
-		(unit 1)
-		(exclude_from_sim no)
-		(in_bom yes)
-		(on_board yes)
-		(dnp no)
-		(property "Reference" "RSW2"
-			(at 456.438 61.976 0)
-			(effects
-				(font
-					(size 1.27 1.27)
-				)
-			)
-		)
-		(property "Value" "RST"
-			(at 452.628 66.802 0)
-			(effects
-				(font
-					(size 1.27 1.27)
-				)
-			)
-		)
-		(property "Footprint" "cornia-footprints:SW_SMD_4x4mm"
-			(at 452.628 64.77 0)
-			(effects
-				(font
-					(size 1.27 1.27)
-				)
-				(hide yes)
-			)
-		)
-		(property "Datasheet" ""
-			(at 452.628 64.77 0)
-			(effects
-				(font
-					(size 1.27 1.27)
-				)
-			)
-		)
-		(property "Description" ""
-			(at 452.628 64.77 0)
-			(effects
-				(font
-					(size 1.27 1.27)
-				)
-				(hide yes)
-			)
-		)
-		(pin "1"
-		)
-		(pin "2"
-		)
-		(instances
-			(project "chocofi"
-				(path "/4976ae50-9ae0-4449-9f0b-b92cb3fc915b"
-					(reference "RSW2")
-					(unit 1)
-				)

Commit message: wip
Parts:
- removed F1, F2, F3: Conn_01x02_Pin, Switches_Chukozor:soldering-pull_switch_Only_Left, symbol Connector:Conn_01x02_Pin
- removed FF1: Conn_01x02_Pin, Switches_Chukozor:soldering-pull_switch, symbol Connector:Conn_01x02_Pin
- added F1, F2, F3, FF1: Conn_01x04, symbol Chukozor_symbols:Conn_01x04
- KLow-1: footprint FPC_connectors_Chukozor:FPC_8pins_687108183722_reversible-Mobile-IN-LOW-V2 -> FPC_connectors_Chukozor:FPC_8pins_687108183722_reversible-Mobile-IN-LOW-FROMBELOW
- KLow-2: footprint FPC_connectors_Chukozor:FPC_8pins_687108183722_reversible-Mobile-IN-LOW-V2 -> FPC_connectors_Chukozor:FPC_8pins_687108183722_reversible-Mobile-IN-TOPP-FROMBELOW
Connections:
- net col0: now also F1.1 (Pin_4)
- net col2: now also F3.1 (Pin_4)
- net row3: now also F1.4 (Pin_1), F2.4 (Pin_1), F3.4 (Pin_1)
- net at Pull1.1: now also FF1.1 (Pin_4)
- net at D33.1 (K): now also FF1.4 (Pin_1)
- no-connect marks 31 -> 39
Other:
- moved on the sheet: Flick3, KLow-2

Commit message: wip
Parts:
- F1, F2, F3, FF1: footprint (none) -> FPC_connectors_Chukozor:FPC_4pins_VERTICAL_MOUSER-FFC2A3308TR-OUT-routed
Changed lines of the file:
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@@
 			)
 		)
-		(property "Footprint" ""
+		(property "Footprint" "FPC_connectors_Chukozor:FPC_4pins_VERTICAL_MOUSER-FFC2A3308TR-OUT-routed"
 			(at 52.832 466.598 0)
 			(effects
@@
 			)
 		)
-		(property "Footprint" ""
+		(property "Footprint" "FPC_connectors_Chukozor:FPC_4pins_VERTICAL_MOUSER-FFC2A3308TR-OUT-routed"
 			(at 109.982 377.444 0)
 			(effects
@@
 			)
 		)
-		(property "Footprint" ""
+		(property "Footprint" "FPC_connectors_Chukozor:FPC_4pins_VERTICAL_MOUSER-FFC2A3308TR-OUT-routed"
 			(at 150.368 377.444 0)
 			(effects
@@
 			)
 		)
-		(property "Footprint" ""
+		(property "Footprint" "FPC_connectors_Chukozor:FPC_4pins_VERTICAL_MOUSER-FFC2A3308TR-OUT-routed"
 			(at 68.58 377.444 0)
 			(effects

Commit message: wip
Parts:
- F1, F2, F3, FF1: footprint FPC_connectors_Chukozor:FPC_4pins_VERTICAL_MOUSER-FFC2A3308TR-OUT-routed -> FPC_connectors_Chukozor:FPC_4pins_Horizontal-PULL-IN-AND-OUT
Connections:
- net at FF1.1 (Pin_4): now also D33.1 (K); no longer Pull1.1
- net at FF1.4 (Pin_1): now also Pull1.1; no longer D33.1 (K)
Other:
- moved on the sheet: FF1
Changed lines of the file:
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@@
 	(symbol
 		(lib_id "Chukozor_symbols:Conn_01x04")
-		(at 52.832 466.598 270)
+		(at 50.292 466.598 90)
+		(mirror x)
 		(unit 1)
 		(exclude_from_sim no)
@@
 			)
 		)
-		(property "Footprint" "FPC_connectors_Chukozor:FPC_4pins_VERTICAL_MOUSER-FFC2A3308TR-OUT-routed"
-			(at 52.832 466.598 0)
+		(property "Footprint" "FPC_connectors_Chukozor:FPC_4pins_Horizontal-PULL-IN-AND-OUT"
+			(at 50.292 466.598 0)
 			(effects
 				(font
@@
 		)
 		(property "Datasheet" "~"
-			(at 52.832 466.598 0)
+			(at 50.292 466.598 0)
 			(effects
 				(font
@@
 		)
 		(property "Description" "Generic connector, single row, 01x04, script generated (kicad-library-utils/schlib/autogen/connector/)"
-			(at 52.832 466.598 0)
+			(at 50.292 466.598 0)
 			(effects
 				(font
@@
 			)
 		)
-		(property "Footprint" "FPC_connectors_Chukozor:FPC_4pins_VERTICAL_MOUSER-FFC2A3308TR-OUT-routed"
+		(property "Footprint" "FPC_connectors_Chukozor:FPC_4pins_Horizontal-PULL-IN-AND-OUT"
 			(at 109.982 377.444 0)
 			(effects
@@
 			)
 		)
-		(property "Footprint" "FPC_connectors_Chukozor:FPC_4pins_VERTICAL_MOUSER-FFC2A3308TR-OUT-routed"
+		(property "Footprint" "FPC_connectors_Chukozor:FPC_4pins_Horizontal-PULL-IN-AND-OUT"
 			(at 150.368 377.444 0)
 			(effects
@@
 			)
 		)
-		(property "Footprint" "FPC_connectors_Chukozor:FPC_4pins_VERTICAL_MOUSER-FFC2A3308TR-OUT-routed"
+		(property "Footprint" "FPC_connectors_Chukozor:FPC_4pins_Horizontal-PULL-IN-AND-OUT"
 			(at 68.58 377.444 0)
 			(effects

Commit message: wip
Parts:
- Pull1: footprint Switches_Chukozor:Kailh_socket_PG1350_reversible_Chukozor_-PULL -> Switches_Chukozor:Kailh_socket_PG1350_reversible_Chukozor_-PULL-simplifie
Changed lines of the file:
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@@
 			)
 		)
-		(property "Footprint" "Switches_Chukozor:Kailh_socket_PG1350_reversible_Chukozor_-PULL"
+		(property "Footprint" "Switches_Chukozor:Kailh_socket_PG1350_reversible_Chukozor_-PULL-simplifie"
 			(at 51.308 452.882 0)
 			(effects
